File: pcb_assignment/pcb_assignment.kicad_sch (KiCad schematic)
At the start: 3 parts, among them SW1 SW_Push

Commit message: donezo2
Parts:
- added R1: 500, symbol Device:R
Connections:
- net at A1.2 (3V3), SW1.1: no longer PS1.4 (+Vo)
- net at A1.28 (VBAT): now also PS1.4 (+Vo)
- net at A1.4 (GND), PS1.3 (-Vo): now also R1.2; no longer SW1.2
- net at A1.9 (IO36/A4): now also SW1.2, R1.1
Other:
- moved on the sheet: SW1
Changed lines of the file:
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@@
 	)
 	(junction
-		(at 153.67 76.2)
+		(at 185.42 115.57)
 		(diameter 0)
 		(color 0 0 0 0)
 	)
+	(junction
+		(at 185.42 143.51)
+		(diameter 0)
+		(color 0 0 0 0)
+	)
+	(wire
+		(pts
+			(xy 185.42 109.22) (xy 185.42 115.57)
+		)
+		(stroke
+			(width 0)
+			(type default)
+		)
+	)
+	(wire
+		(pts
+			(xy 185.42 123.19) (xy 185.42 143.51)
+		)
+		(stroke
+			(width 0)
+			(type default)
+		)
+	)
 	(wire
 		(pts
@@
 	(wire
 		(pts
-			(xy 186.69 143.51) (xy 151.13 143.51)
+			(xy 186.69 143.51) (xy 185.42 143.51)
+		)
+		(stroke
+			(width 0)
+			(type default)
+		)
+	)
+	(wire
+		(pts
+			(xy 163.83 115.57) (xy 185.42 115.57)
 		)
 		(stroke
@@
 	(wire
 		(pts
-			(xy 176.53 76.2) (xy 176.53 85.09)
+			(xy 185.42 81.28) (xy 176.53 81.28)
+		)
+		(stroke
+			(width 0)
+			(type default)
+		)
+	)
+	(wire
+		(pts
+			(xy 176.53 76.2) (xy 176.53 81.28)
+		)
+		(stroke
+			(width 0)
+			(type default)
+		)
+	)
+	(wire
+		(pts
+			(xy 118.11 59.69) (xy 148.59 59.69)
 		)
 		(stroke
@@
 	(wire
 		(pts
-			(xy 153.67 59.69) (xy 153.67 76.2)
-		)
-		(stroke
-			(width 0)
-			(type default)
-		)
-	)
-	(wire
-		(pts
-			(xy 118.11 59.69) (xy 153.67 59.69)
-		)
-		(stroke
-			(width 0)
-			(type default)
-		)
-	)
-	(wire
-		(pts
-			(xy 186.69 85.09) (xy 186.69 143.51)
+			(xy 148.59 59.69) (xy 148.59 80.01)
 		)
 		(stroke
@@
 	(wire
 		(pts
+			(xy 185.42 143.51) (xy 151.13 143.51)
+		)
+		(stroke
+			(width 0)
+			(type default)
+		)
+	)
+	(wire
+		(pts
 			(xy 97.79 66.04) (xy 97.79 64.77)
 		)
@@
 		(pts
 			(xy 78.74 66.04) (xy 97.79 66.04)
+		)
+		(stroke
+			(width 0)
+			(type default)
+		)
+	)
+	(wire
+		(pts
+			(xy 185.42 99.06) (xy 185.42 81.28)
 		)
 		(stroke
@@
 				(justify left)
 				(hide yes)
+			)
+		)
+	)
+	(symbol
+		(lib_id "Device:R")
+		(at 185.42 119.38 0)
+		(unit 1)
+		(exclude_from_sim no)
+		(in_bom yes)
+		(on_board yes)
+		(dnp no)
+		(fields_autoplaced yes)
+		(property "Reference" "R1"
+			(at 187.96 118.1099 0)
+			(effects
+				(font
+					(size 1.27 1.27)
+				)
+				(justify left)
+			)
+		)
+		(property "Value" "500"
+			(at 187.96 120.6499 0)
+			(effects
+				(font
+					(size 1.27 1.27)
+				)
+				(justify left)
+			)
+		)
+		(property "Footprint" ""
+			(at 183.642 119.38 90)
+			(effects
+				(font
+					(size 1.27 1.27)
+				)
+				(hide yes)
+			)
+		)
+		(property "Datasheet" "~"
+			(at 185.42 119.38 0)
+			(effects
+				(font
+					(size 1.27 1.27)
+				)
+				(hide yes)
+			)
+		)
+		(property "Description" "Resistor"
+			(at 185.42 119.38 0)
+			(effects
+				(font
+					(size 1.27 1.27)
+				)
+				(hide yes)
+			)
+		)
+		(pin "2"
+		)
+		(pin "1"
+		)
+		(instances
+			(project "pcb_assignment"
+				(path "/925b6437-be0e-45b6-a75c-5b5ce07134fb"
+					(reference "R1")
+					(unit 1)
+				)
 			)
 		)
@@
 	(symbol
 		(lib_id "Switch:SW_Push")
-		(at 181.61 85.09 0)
+		(at 185.42 104.14 270)
 		(unit 1)
 		(exclude_from_sim no)
@@
 		(fields_autoplaced yes)
 		(property "Reference" "SW1"
-			(at 181.61 77.47 0)
-			(effects
-				(font
-					(size 1.27 1.27)
-				)
+			(at 189.23 102.8699 90)
+			(effects
+				(font
+					(size 1.27 1.27)
+				)
+				(justify left)
 			)
 		)
 		(property "Value" "SW_Push"
-			(at 181.61 80.01 0)
-			(effects
-				(font
-					(size 1.27 1.27)
-				)
+			(at 189.23 105.4099 90)
+			(effects
+				(font
+					(size 1.27 1.27)
+				)
+				(justify left)
 			)
 		)
 		(property "Footprint" ""
-			(at 181.61 80.01 0)
+			(at 190.5 104.14 0)
 			(effects
 				(font
@@
 		)
 		(property "Datasheet" "~"
-			(at 181.61 80.01 0)
+			(at 190.5 104.14 0)
 			(effects
 				(font
@@
 		)
 		(property "Description" "Push button switch, generic, two pins"
-			(at 181.61 85.09 0)
-			(effects
-				(font
+			(at 185.42 104.14 0)
+			(effects
+				(font

Commit message: all bueno
Parts:
- removed A1: Adafruit_Feather_HUZZAH32_ESP32, Module:Adafruit_Feather, symbol MCU_Module:Adafruit_Feather_HUZZAH32_ESP32
- removed PS1: IRM-20-5, Converter_ACDC:Converter_ACDC_MeanWell_IRM-20-xx_THT, symbol Converter_ACDC:IRM-20-5
- removed R1: 500, symbol Device:R
- removed SW1: SW_Push, symbol Switch:SW_Push
- added BZ1: Buzzer, Buzzer_Beeper:Buzzer_15x7.5RM7.6, symbol Device:Buzzer
- added R2: 200, Resistor_THT:R_Axial_DIN0207_L6.3mm_D2.5mm_P7.62mm_Horizontal, symbol Device:R
- added R3: 1k, Resistor_THT:R_Axial_DIN0207_L6.3mm_D2.5mm_P15.24mm_Horizontal, symbol Device:R
- added SW2: SW_Push, Button_Switch_SMD:SW_Push_1P1T_NO_6x6mm_H9.5mm, symbol Switch:SW_Push
- added Xiao1: ~, xiao ESP32S3_PCB:MOUDLE14P-SMD-2.54-21X17.8MM, symbol 196ece:xiaos3sense
Connections:
- new net: BZ1.1 (+), Xiao1.1 (D0)
- new net: BZ1.2 (-), R2.1
- new net: SW2.1, Xiao1.12 (3V3)
- new net: R3.1, SW2.2, Xiao1.9 (D8)
- new net: R2.2, R3.2, Xiao1.13 (GND)
